Commit message: extended orange block in URDF

File: urdf/ur5.urdf (robot description, URDF)
Before this commit: robot universal_robot, 9 links, 8 joints
Links:
- link ee_link: geometry collision box size=0.12 0.01 0.01

Commit message: shortned extra pipe length

File: urdf/ur5.urdf (robot description, URDF)
Before this commit: robot universal_robot, 9 links, 8 joints
Links:
- link ee_link: geometry collision box size=0.08 0.01 0.01
